File: Ethernet/eth_rj45-sma/eth_rj45-sma.kicad_pcb (KiCad board)
At the start: 2 copper layers, 198.8 x 124.8 mm, 48 parts, among them J1 RJ45, J10 TX+, J11 TX-, J12 TX+, J13 TX-, J14 TX+, J15 TX-, J16 RX+, J17 RX-, J18 RX-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

Commit message: ProgressWithAnOtherCircuit
Parts:
- R1, R11, R12, R13, R14, R2, R3, R4: footprint Resistor_SMD:R_0603_1608Metric_Pad1.05x0.95mm_HandSolder -> Resistor_SMD:R_1206_3216Metric_Pad1.42x1.75mm_HandSolder
- moved R13 17.5 mm to (208.0, 140.5), turned to 270 degrees
- moved R14 11.1 mm to (210.6, 140.5), turned to 270 degrees
Routing:
- net Net-(R13-Pad1): track 2.17 -> 21.0 mm, vias 0 -> 2
- net Net-(R14-Pad1): track 2.17 -> 11.8 mm, vias 0 -> 2
- net Net-(J9-Pad6): track 14.0 -> 13.4 mm
- net GND: vias 42 -> 41
