File: Ethernet/eth_rj45-sma/eth_rj45-sma.sch (KiCad schematic (older format))
At the start: 22 parts

Commit message: Eth-RJ45_adapters_complete
Parts:
- added C1, C2, C3, C4: 100n, Capacitor_SMD:C_0603_1608Metric_Pad1.05x0.95mm_HandSolder, symbol Device:C
- added J10, J14: TX+, Connector_Coaxial:SMA_Amphenol_132289_EdgeMount, symbol Connector:Conn_Coaxial
- added J11, J15: TX-, Connector_Coaxial:SMA_Amphenol_132289_EdgeMount, symbol Connector:Conn_Coaxial
- added J12: TX+, Connector_Coaxial:SMA_Amphenol_132134_Vertical, symbol Connector:Conn_Coaxial
- added J13: TX-, Connector_Coaxial:SMA_Amphenol_132134_Vertical, symbol Connector:Conn_Coaxial
- added J16, J24: RX+, Connector_Coaxial:SMA_Amphenol_132289_EdgeMount, symbol Connector:Conn_Coaxial
- added J17, J25: RX-, Connector_Coaxial:SMA_Amphenol_132289_EdgeMount, symbol Connector:Conn_Coaxial
- added J18: RX-, Connector_Coaxial:SMA_Amphenol_132134_Vertical, symbol Connector:Conn_Coaxial
- added J19: RX+, Connector_Coaxial:SMA_Amphenol_132134_Vertical, symbol Connector:Conn_Coaxial
- added J7: TX, Connector_Coaxial:SMA_Amphenol_132134_Vertical, symbol Connector:Conn_Coaxial
- added J8: RX, Connector_Coaxial:SMA_Amphenol_132134_Vertical, symbol Connector:Conn_Coaxial
- added R1, R3: 75R, Resistor_SMD:R_0603_1608Metric_Pad1.05x0.95mm_HandSolder, symbol Device:R
- added R10, R9: 0R, Resistor_SMD:R_0603_1608Metric_Pad1.05x0.95mm_HandSolder, symbol Device:R
- added R5, R6, R7, R8: 50R, Resistor_SMD:R_0603_1608Metric_Pad1.05x0.95mm_HandSolder, symbol Device:R
- C5, C6: renamed from C?; value C -> 10n; footprint (none) -> Capacitor_SMD:C_0603_1608Metric_Pad1.05x0.95mm_HandSolder
- J1, J2, J9: renamed from J?; footprint (none) -> Connector_RJ:RJ45_Ninigi_GE; symbol Connector:RJ45 -> Connector:8P8C_Shielded
- J20, J3: renamed from J?; value Conn_Coaxial -> TX+; footprint (none) -> Connector_Coaxial:SMA_Amphenol_132134_Vertical
- J21, J4: renamed from J?; value Conn_Coaxial -> TX-; footprint (none) -> Connector_Coaxial:SMA_Amphenol_132134_Vertical
- J22, J5: renamed from J?; value Conn_Coaxial -> RX+; footprint (none) -> Connector_Coaxial:SMA_Amphenol_132134_Vertical
- J23, J6: renamed from J?; value Conn_Coaxial -> RX-; footprint (none) -> Connector_Coaxial:SMA_Amphenol_132134_Vertical
- R11, R12, R13, R14, R2, R4: renamed from R?; footprint (none) -> Resistor_SMD:R_0603_1608Metric_Pad1.05x0.95mm_HandSolder
- gave numbers to parts that had none: 3
Connections:
- net at J2.4: now also J2.5, R4.1
- net at J2.7: now also J2.8, R2.1
- net at J9.4: now also J9.5, R12.1
- net at J9.7: now also J9.8, R11.1
- net GND: now reaches J3.2 (Ext)
- net GND: now also C5.2, C6.2, J1.SH, J2.SH, J20.2 (Ext), J21.2 (Ext), J22.2 (Ext), J23.2 (Ext), J4.2 (Ext), J5.2 (Ext), J6.2 (Ext), J9.SH, R11.2, R12.2, R13.2, R14.2, R2.2, R4.2, TR1.6, TR2.6, J10.2 (Ext), J11.2 (Ext), J12.2 (Ext), J13.2 (Ext), J14.2 (Ext), J15.2 (Ext), J16.2 (Ext), J17.2 (Ext), J18.2 (Ext), J19.2 (Ext), J24.2 (Ext), J25.2 (Ext), J7.2 (Ext), J8.2 (Ext), R1.2, R10.1, R3.2, R9.1
- net at TR3.10 (C_RX): now also C5.1
- net at TR3.15 (C_TX): now also C6.1
- net at TR3.2 (C_TD): now also R13.1
- net at TR3.7 (C_RD): now also R14.1
- net at TR1.1: now also C2.1
- net at TR1.3: now also C1.1
- net at TR1.4: now also J7.1 (In)
- net at TR2.1: now also C4.1
- net at TR2.3: now also C3.1
- net at TR2.4: now also J8.1 (In)
- net at J1.1: now also C1.2, R5.1
- net at J1.2: now also C2.2, R6.2
- net at J1.3: now also C3.2, R7.1
- net at J1.4: now also J1.5, R3.1
- net at J1.6: now also C4.2, R8.2
- net at J1.7: now also J1.8, R1.1
- new net: J10.1 (In), J12.1 (In), J14.1 (In)
- new net: J11.1 (In), J13.1 (In), J15.1 (In)
- new net: J16.1 (In), J19.1 (In), J24.1 (In)
- new net: J17.1 (In), J18.1 (In), J25.1 (In)
- new net: R5.2, R6.1, R9.2
- new net: R10.2, R7.2, R8.1
Other:
- note added: "100Base-TX\nmeasurement"
- note added: "RJ45-SMA balun\nboard"
- note added: "RJ45-SMA with magnetics\nboard"
- note added: "RJ45-SMA\nboard"
- moved on the sheet: C5, C6, J20, J21, J22, J23, J3, J4, J5, J6, R11, R12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

Commit message: ProgressWithAnOtherCircuit
Parts:
- R1, R11, R12, R13, R14, R2, R3, R4: footprint Resistor_SMD:R_0603_1608Metric_Pad1.05x0.95mm_HandSolder -> Resistor_SMD:R_1206_3216Metric_Pad1.42x1.75mm_HandSolder
Changed lines of the file:
@@
 F 0 "R11" H 7070 2446 50  0000 L CNN
 F 1 "75R" H 7070 2355 50  0000 L CNN
-F 2 "Resistor_SMD:R_0603_1608Metric_Pad1.05x0.95mm_HandSolder" V 6930 2400 50  0001 C CNN
+F 2 "Resistor_SMD:R_1206_3216Metric_Pad1.42x1.75mm_HandSolder" V 6930 2400 50  0001 C CNN
 F 3 "~" H 7000 2400 50  0001 C CNN
 	1    7000 2400
@@
 F 0 "R12" H 7345 2446 50  0000 L CNN
 F 1 "75R" H 7345 2355 50  0000 L CNN
-F 2 "Resistor_SMD:R_0603_1608Metric_Pad1.05x0.95mm_HandSolder" V 7205 2400 50  0001 C CNN
+F 2 "Resistor_SMD:R_1206_3216Metric_Pad1.42x1.75mm_HandSolder" V 7205 2400 50  0001 C CNN
 F 3 "~" H 7275 2400 50  0001 C CNN
 	1    7275 2400
@@
 F 0 "R13" H 7620 2446 50  0000 L CNN
 F 1 "75R" H 7620 2355 50  0000 L CNN
-F 2 "Resistor_SMD:R_0603_1608Metric_Pad1.05x0.95mm_HandSolder" V 7480 2400 50  0001 C CNN
+F 2 "Resistor_SMD:R_1206_3216Metric_Pad1.42x1.75mm_HandSolder" V 7480 2400 50  0001 C CNN
 F 3 "~" H 7550 2400 50  0001 C CNN
 	1    7550 2400
@@
 F 0 "R14" H 7895 2446 50  0000 L CNN
 F 1 "75R" H 7895 2355 50  0000 L CNN
-F 2 "Resistor_SMD:R_0603_1608Metric_Pad1.05x0.95mm_HandSolder" V 7755 2400 50  0001 C CNN
+F 2 "Resistor_SMD:R_1206_3216Metric_Pad1.42x1.75mm_HandSolder" V 7755 2400 50  0001 C CNN
 F 3 "~" H 7825 2400 50  0001 C CNN
 	1    7825 2400
@@
 F 0 "R2" H 1970 2246 50  0000 L CNN
 F 1 "75R" H 1970 2155 50  0000 L CNN
-F 2 "Resistor_SMD:R_0603_1608Metric_Pad1.05x0.95mm_HandSolder" V 1830 2200 50  0001 C CNN
+F 2 "Resistor_SMD:R_1206_3216Metric_Pad1.42x1.75mm_HandSolder" V 1830 2200 50  0001 C CNN
 F 3 "~" H 1900 2200 50  0001 C CNN
 	1    1900 2200
@@
 F 0 "R4" H 2245 2246 50  0000 L CNN
 F 1 "75R" H 2245 2155 50  0000 L CNN
-F 2 "Resistor_SMD:R_0603_1608Metric_Pad1.05x0.95mm_HandSolder" V 2105 2200 50  0001 C CNN
+F 2 "Resistor_SMD:R_1206_3216Metric_Pad1.42x1.75mm_HandSolder" V 2105 2200 50  0001 C CNN
 F 3 "~" H 2175 2200 50  0001 C CNN
 	1    2175 2200
@@
 F 0 "R3" H 2045 6146 50  0000 L CNN
 F 1 "75R" H 2045 6055 50  0000 L CNN
-F 2 "Resistor_SMD:R_0603_1608Metric_Pad1.05x0.95mm_HandSolder" V 1905 6100 50  0001 C CNN
+F 2 "Resistor_SMD:R_1206_3216Metric_Pad1.42x1.75mm_HandSolder" V 1905 6100 50  0001 C CNN
 F 3 "~" H 1975 6100 50  0001 C CNN
 	1    1975 6100
@@
 F 0 "R1" H 1770 6121 50  0000 L CNN
 F 1 "75R" H 1770 6030 50  0000 L CNN
-F 2 "Resistor_SMD:R_0603_1608Metric_Pad1.05x0.95mm_HandSolder" V 1630 6075 50  0001 C CNN
+F 2 "Resistor_SMD:R_1206_3216Metric_Pad1.42x1.75mm_HandSolder" V 1630 6075 50  0001 C CNN
 F 3 "~" H 1700 6075 50  0001 C CNN
 	1    1700 6075
