File: Ethernet/eth_phy_KSZ8041MLL_poe/eth_phy_KSZ8041MLL_poe.kicad_pcb (KiCad board)
At the start: 2 copper layers, 90 x 60 mm, 44 parts, among them IC1 KSZ8041MLL, J1 Conn_02x12_Odd_Even, J2 ARJM11D7-114-AB-EW2, J3 Conn_Coaxial, X1 ECS-2520MV-xxx-xx

Commit message: SomeBoardsReady
Parts:
- added H1: MountingHole, MountingHole:MountingHole_3.2mm_M3_Pad_Via, F.Cu at (192.0, 57.0)
- added H2: MountingHole, MountingHole:MountingHole_3.2mm_M3_Pad_Via, F.Cu at (114.0, 105.0)
- added H3: MountingHole, MountingHole:MountingHole_3.2mm_M3_Pad_Via, F.Cu at (192.0, 105.0)
- added H4: MountingHole, MountingHole:MountingHole_3.2mm_M3_Pad_Via, F.Cu at (114.0, 57.0)
- C11, C13: value 10n -> 10u
Connections:
- C11 pad 1: Net-(C11-Pad1) -> /A3V3
- C13 pad 1: Net-(C13-Pad1) -> /A3V3
- IC1 pad 14: Net-(IC1-Pad14) -> (no net)
- IC1 pad 44: Net-(IC1-Pad44) -> (no net)
- IC1 pad 45: Net-(IC1-Pad45) -> (no net)
- IC1 pad 46: Net-(IC1-Pad46) -> (no net)
- IC1 pad 48: Net-(IC1-Pad48) -> (no net)
- J2 pad 4: Net-(C13-Pad1) -> /A3V3
- J2 pad 9: Net-(C11-Pad1) -> /A3V3
- J2 pad SH: GND -> (no net)
Routing:
- net /A3V3: track 21.4 -> 99.3 mm, vias 1 -> 3
- net Net-(C11-Pad1): track 13.4 -> 0.00 mm
- net Net-(C13-Pad1): track 11.0 -> 0.00 mm
- net /3V3: track 272.5 -> 271.5 mm
- net GND: vias 67 -> 71
