File: Ethernet/eth_phy_KSZ8041MLL_mezzanine/eth_phy_KSZ8041MLL_mezzanine.kicad_pcb (KiCad board)
At the start: 2 copper layers, 90 x 60 mm, 40 parts, among them IC1 KSZ8041MLL, J1 Conn_02x12_Odd_Even, J2 Conn_01x09_Female, X1 ECS-2520MV-xxx-xx

Commit message: FirstRoundPanelsDone
Parts:
- added C15: 10u, Capacitor_SMD:C_0805_2012Metric_Pad1.18x1.45mm_HandSolder, F.Cu at (130.4, 123.5)
- added D4: LED, LED_SMD:LED_0805_2012Metric_Pad1.15x1.40mm_HandSolder, F.Cu at (140.0, 127.4)
- added D5: LED, LED_SMD:LED_0805_2012Metric_Pad1.15x1.40mm_HandSolder, F.Cu at (140.0, 119.9)
- added R1: 4k7, Resistor_SMD:R_0805_2012Metric_Pad1.20x1.40mm_HandSolder, F.Cu at (134.5, 127.4)
- added R2: 470, Resistor_SMD:R_0805_2012Metric_Pad1.20x1.40mm_HandSolder, F.Cu at (134.6, 124.9)
- added R3: 4k7, Resistor_SMD:R_0805_2012Metric_Pad1.20x1.40mm_HandSolder, F.Cu at (134.5, 119.9)
- added R4: 470, Resistor_SMD:R_0805_2012Metric_Pad1.20x1.40mm_HandSolder, F.Cu at (134.5, 122.4)
- moved H6 22.0 mm to (152.1, 117.6)
- moved H5 18.3 mm to (152.1, 91.8)
- moved J2 18.1 mm to (158.5, 104.7)
- moved C11 9.84 mm to (141.4, 113.8), turned to 270 degrees
- moved C13 5.06 mm to (151.0, 106.7), turned to 180 degrees
Connections:
- IC1 pad 42: (no net) -> /LED0
- IC1 pad 43: (no net) -> /LED1
Routing:
- net (no net): track 100.7 -> 0.00 mm, vias 2 -> 0
- net /TX+: track 3.27 -> 57.3 mm
- net /TX-: track 5.13 -> 59.1 mm
- net /RX-: track 6.85 -> 43.1 mm
- net /RX+: track 8.42 -> 44.7 mm
- net /LED0: track 0.00 -> 32.6 mm, vias 0 -> 2
- net /3V3: track 234.9 -> 205.5 mm
- net /LED1: track 0.00 -> 25.2 mm, vias 0 -> 2
- net /A3V3: track 42.7 -> 52.0 mm
- net Net-(D5-Pad2): track 0.00 -> 7.30 mm
- net Net-(D4-Pad2): track 0.00 -> 7.18 mm
- net GND: vias 45 -> 111
