File: Ethernet/eth_phy_KSZ8041MLL_mezzanine/eth_phy_KSZ8041MLL_mezzanine.sch (KiCad schematic (older format))
At the start: 44 parts, among them IC1 KSZ8041MLL, J1 Conn_02x12_Odd_Even, J2 ARJM11D7-114-AB-EW2, J3 Conn_Coaxial, X1 ECS-2520MV-xxx-xx

Commit message: SomeBoardsReady
Parts:
- removed C15: 1n / 2000V, Capacitor_SMD:C_1206_3216Metric_Pad1.42x1.75mm_HandSolder, symbol Device:C
- removed C16, C18: 1u, Capacitor_SMD:C_0603_1608Metric_Pad1.08x0.95mm_HandSolder, symbol Device:C
- removed J2: ARJM11D7-114-AB-EW2, myfootprintlib:ARJM11D7-114-AB-EW2, symbol myethlibopen:ARJM11D7-114-AB-EW2
- removed J3: Conn_Coaxial, Connector_Coaxial:BNC_TEConnectivity_1478204_Vertical, symbol Connector:Conn_Coaxial
- removed R1, R2: 75R, Resistor_SMD:R_0603_1608Metric_Pad1.05x0.95mm_HandSolder, symbol Device:R
- removed R3, R5: 4k7, Resistor_SMD:R_0603_1608Metric_Pad1.05x0.95mm_HandSolder, symbol Device:R
- removed R4, R6: 470R, Resistor_SMD:R_0603_1608Metric_Pad1.05x0.95mm_HandSolder, symbol Device:R
- added H1, H2, H3, H4: MountingHole, MountingHole:MountingHole_3.2mm_M3_Pad_Via, symbol Mechanical:MountingHole
- added H5, H6: MountingHole_Pad, MountingHole:MountingHole_3.2mm_M3_Pad_Via, symbol Mechanical:MountingHole_Pad
- added J2: Conn_01x09_Female, myfootprintlib:mezzanine_9p_10162582-1134109LF_Conan_1mm, symbol Connector:Conn_01x09_Female
Connections:
- net labels removed: GNDIN, PWRIN
- wire segments 262 -> 233

Commit message: FirstRoundPanelsDone
Parts:
- added C15: 10u, Capacitor_SMD:C_0805_2012Metric_Pad1.18x1.45mm_HandSolder, symbol Device:C
- added D4, D5: LED, LED_SMD:LED_0805_2012Metric_Pad1.15x1.40mm_HandSolder, symbol Device:LED
- added R1, R3: 4k7, Resistor_SMD:R_0805_2012Metric_Pad1.20x1.40mm_HandSolder, symbol Device:R
- added R2, R4: 470, Resistor_SMD:R_0805_2012Metric_Pad1.20x1.40mm_HandSolder, symbol Device:R
Connections:
- net 3V3: now also C15.1, R1.1, R2.1, R3.1, R4.1
- net GND: now also C15.2
- net LED0: now also D4.1 (K), R1.2
- net LED1: now also D5.1 (K), R3.2
- new net: D4.2 (A), R2.2
- new net: D5.2 (A), R4.2
Changed lines of the file:
@@
 Wire Wire Line
 	9875 1175 10250 1175
+$Comp
+L Device:R R2
+U 1 1 61C08698
+P 9925 2400
+F 0 "R2" H 9995 2446 50  0000 L CNN
+F 1 "470" H 9995 2355 50  0000 L CNN
+F 2 "Resistor_SMD:R_0805_2012Metric_Pad1.20x1.40mm_HandSolder" V 9855 2400 50  0001 C CNN
+F 3 "~" H 9925 2400 50  0001 C CNN
+	1    9925 2400
+	1    0    0    -1
+$EndComp
+$Comp
+L Device:R R4
+U 1 1 61C08C4C
+P 10475 2400
+F 0 "R4" H 10545 2446 50  0000 L CNN
+F 1 "470" H 10545 2355 50  0000 L CNN
+F 2 "Resistor_SMD:R_0805_2012Metric_Pad1.20x1.40mm_HandSolder" V 10405 2400 50  0001 C CNN
+F 3 "~" H 10475 2400 50  0001 C CNN
+	1    10475 2400
+	1    0    0    -1
+$EndComp
+$Comp
+L Device:R R1
+U 1 1 61C08E32
+P 9650 2400
+F 0 "R1" H 9720 2446 50  0000 L CNN
+F 1 "4k7" H 9720 2355 50  0000 L CNN
+F 2 "Resistor_SMD:R_0805_2012Metric_Pad1.20x1.40mm_HandSolder" V 9580 2400 50  0001 C CNN
+F 3 "~" H 9650 2400 50  0001 C CNN
+	1    9650 2400
+	1    0    0    -1
+$EndComp
+$Comp
+L Device:R R3
+U 1 1 61C09179
+P 10200 2400
+F 0 "R3" H 10270 2446 50  0000 L CNN
+F 1 "4k7" H 10270 2355 50  0000 L CNN
+F 2 "Resistor_SMD:R_0805_2012Metric_Pad1.20x1.40mm_HandSolder" V 10130 2400 50  0001 C CNN
+F 3 "~" H 10200 2400 50  0001 C CNN
+	1    10200 2400
+	1    0    0    -1
+$EndComp
+$Comp
+L Device:LED D4
+U 1 1 61C0A182
+P 9925 2850
+F 0 "D4" V 9964 2732 50  0000 R CNN
+F 1 "LED" V 9873 2732 50  0000 R CNN
+F 2 "LED_SMD:LED_0805_2012Metric_Pad1.15x1.40mm_HandSolder" H 9925 2850 50  0001 C CNN
+F 3 "~" H 9925 2850 50  0001 C CNN
+	1    9925 2850
+	0    -1   -1   0
+$EndComp
+$Comp
+L Device:LED D5
+U 1 1 61C0AA34
+P 10475 2850
+F 0 "D5" V 10514 2732 50  0000 R CNN
+F 1 "LED" V 10423 2732 50  0000 R CNN
+F 2 "LED_SMD:LED_0805_2012Metric_Pad1.15x1.40mm_HandSolder" H 10475 2850 50  0001 C CNN
+F 3 "~" H 10475 2850 50  0001 C CNN
+	1    10475 2850
+	0    -1   -1   0
+$EndComp
+$Comp
+L Device:C C15
+U 1 1 61C18DE2
+P 9225 2400
+F 0 "C15" H 9340 2446 50  0000 L CNN
+F 1 "10u" H 9340 2355 50  0000 L CNN
+F 2 "Capacitor_SMD:C_0805_2012Metric_Pad1.18x1.45mm_HandSolder" H 9263 2250 50  0001 C CNN
+F 3 "~" H 9225 2400 50  0001 C CNN
+	1    9225 2400
+	1    0    0    -1
+$EndComp
+Wire Wire Line
+	10475 2250 10475 2075
+Wire Wire Line
+	10475 2075 10200 2075
+Wire Wire Line
+	9225 2250 9225 2075
+Connection ~ 9225 2075
+Wire Wire Line
+	9225 2075 8625 2075
+Wire Wire Line
+	9650 2250 9650 2075
+Connection ~ 9650 2075
+Wire Wire Line
+	9650 2075 9225 2075
+Wire Wire Line
+	9925 2250 9925 2075
+Connection ~ 9925 2075
+Wire Wire Line
+	9925 2075 9650 2075
+Connection ~ 10200 2075
+Wire Wire Line
+	10200 2075 9925 2075
+Wire Wire Line
+	10200 2075 10200 2250
+Wire Wire Line
+	9925 2550 9925 2700
+Wire Wire Line
+	10475 2550 10475 2700
+Wire Wire Line
+	9925 3000 9925 3150
+Wire Wire Line
+	9925 3150 9650 3150
+Wire Wire Line
+	10475 3000 10475 3300
+Wire Wire Line
+	10475 3300 10200 3300
+Wire Wire Line
+	9650 2550 9650 3150
+Connection ~ 9650 3150
+Wire Wire Line
+	9650 3150 9325 3150
+Wire Wire Line
+	10200 2550 10200 3300
+Connection ~ 10200 3300
+Wire Wire Line
+	10200 3300 9325 3300
+$Comp
+L power:GND #PWR0107
+U 1 1 61CD1C00
+P 9225 2700
+F 0 "#PWR0107" H 9225 2450 50  0001 C CNN
+F 1 "GND" H 9230 2527 50  0000 C CNN
+F 2 "" H 9225 2700 50  0001 C CNN
+F 3 "" H 9225 2700 50  0001 C CNN
+	1    9225 2700
+	1    0    0    -1
+$EndComp
+Wire Wire Line
+	9225 2550 9225 2700
+Text Label 8625 2075 0    50   ~ 0
+3V3
+Text Label 9325 3150 0    50   ~ 0
+LED0
+Text Label 9325 3300 0    50   ~ 0
+LED1
 $EndSCHEMATC
